Commit message: controller manager working

File: robotic_arm_pkg/urdf/arm_meshed.urdf (robot description, URDF)
Before this commit: robot arm_mesh, 8 links, 7 joints
Links:
- removed link claw_L
- removed link claw_R
Joints:
- removed joint gripper_base_claw_L
- removed joint gripper_base_claw_R

Commit message: moveit integration with hardware_interface

File: robotic_arm_pkg/urdf/arm_meshed.urdf (robot description, URDF)
Before this commit: robot arm_mesh, 6 links, 5 joints
Links:
- added link claw_L, mass 0.007; collision mesh filename=package://robotic_arm_pkg/meshes/gripper_claw_L.stl scale=0.001 0.001 0.001; visual mesh filename=package://robotic_arm_pkg/meshes/gripper_claw_L.stl scale=0.001 0.001 0.001
- added link claw_R, mass 0.007; collision mesh filename=package://robotic_arm_pkg/meshes/gripper_claw_R.stl scale=0.001 0.001 0.001; visual mesh filename=package://robotic_arm_pkg/meshes/gripper_claw_R.stl scale=0.001 0.001 0.001
Joints:
- added joint gripper_base_claw_L: type revolute, parent gripper_base, child claw_L, origin xyz=0 -0.0125 0.01 rpy=0 0 0, axis 1 0 0, limit lower=-1.57 upper=1.57 effort=1000.0 velocity=0.5
- added joint gripper_base_claw_R: type revolute, parent gripper_base, child claw_R, origin xyz=0 0.0035 0.012 rpy=0 0 0, axis -1 0 0, limit lower=-1.57 upper=1.57 effort=1000.0 velocity=0.5
